Commit message: xscsdc

File: robot.urdf (robot description, URDF)
Before this commit: robot robot_model, 5 links, 4 joints
Links:
- removed link base_link
- added link base_frame; collision box size=0.20 0.20 0.07; visual box size=0.16 0.16 0.07
Joints:
- joint base_to_rwheel: parent base_link -> base_frame
- joint laser_joint: parent base_link -> base_frame
- joint ultrasonic_joint: parent base_link -> base_frame

Commit message: scvsdv

File: robot.urdf (robot description, URDF)
Before this commit: robot robot_model, 5 links, 4 joints
Joints:
- joint base_to_lwheel: parent base_link -> base_frame
